File: hardware/Ham-ESP32-RPT/Ham-ESP32-RPT.kicad_sch (KiCad schematic)
At the start: 17 parts, among them J1 USB_C_Receptacle_USB2.0_16P, U1 ESP32-S3-WROOM-1, U2 D3V3XA4B10LP, U3 TLV75801PDBV

Commit message: Add BOM to project
Parts:
- removed BOOT1, RESET1: SW_MEC_5E, Button_Switch_SMD:SW_MEC_5GSH9, symbol PCM_Switch:SW_MEC_5E
- added SW1, SW2: SW_SPST, symbol PCM_Switch:SW_SPST
- added U4: CP2104, Package_DFN_QFN:QFN-24-1EP_4x4mm_P0.5mm_EP2.6x2.6mm, symbol Interface_USB:CP2104
Connections:
- net 3V3: no longer C1.1, C2.1, C7.1, R6.1, R8.1, U1.2 (3V3), U3.5 (OUT)
- net ESP32_EN: now also SW2.2 (B)
- net GND: now also SW1.1 (A), SW2.1 (A)
- net at C4.1, U1.27 (IO0): now also SW1.2 (B)
- net 5VUSB renamed +5VP
- new net: U4.2 (GND), U4.25 (GND)
- new net +3.3VP: C1.1, C2.1, C7.1, R6.1, R8.1, U1.2 (3V3), U3.5 (OUT)
