File: hardware/Ham-ESP32-RPT/Ham-ESP32-RPT.kicad_sch (KiCad schematic)
At the start: 21 parts, among them J1 USB_C_Receptacle_USB2.0_16P, J2 Conn_Coaxial, SW1 SW_SPST, SW2 SW_SPST, U1 ESP32-S3-WROOM-1, U2 D3V3XA4B10LP, U3 TLV75801PDBV, U4 CP2104, U4 ESP32-S3-DevKitC

Commit message: Change sound announce
Parts:
- removed SW1, SW2: SW_SPST, symbol PCM_Switch:SW_SPST
- removed U4: CP2104, Package_DFN_QFN:QFN-24-1EP_4x4mm_P0.5mm_EP2.6x2.6mm, symbol Interface_USB:CP2104
- added BOOT1: SW_MEC_5E, Button_Switch_SMD:SW_MEC_5GSH9, symbol PCM_Switch:SW_MEC_5E
Connections:
- net +3.3VP is gone; now on net 3V3: C1.1, C2.1, C7.1, R6.1, R8.1, U1.2 (3V3), U3.5 (OUT)
- net ESP32_EN: now also RESET1.3 (K), RESET1.4 (A)
- net GND: now also RESET1.1, RESET1.2, BOOT1.1, BOOT1.2
- net at C4.1, U1.27 (IO0): now also BOOT1.3 (K), BOOT1.4 (A)
- net +5VP renamed 5VUSB
