File: hardware/Ham-ESP32-RPT/Ham-ESP32-RPT.kicad_pcb (KiCad board)
At the start: 2 copper layers, 100 x 115 mm, 19 parts, among them J1 USB_C_Receptacle_USB2.0_16P, J2 Conn_Coaxial, U1 ESP32-S3-WROOM-1, U2 D3V3XA4B10LP, U3 TLV75801PDBV, U4 ESP32-S3-DevKitC

Commit message: Correct bug for PTT output
Parts:
- moved U4 41.1 mm to (127.0, 99.5), turned to 0 degrees
