File: hardware/Ham-ESP32-RPT/Ham-ESP32-RPT.kicad_pcb (KiCad board)
At the start: 2 copper layers, 66 x 132.5 mm, 17 parts, among them J1 USB_C_Receptacle_USB2.0_16P, U1 ESP32-S3-WROOM-1, U2 D3V3XA4B10LP, U3 TLV75801PDBV

Commit message: Mise à jour de la documentation
Parts:
- moved R3 40.3 mm to (133.4, 54.5)
- moved C3 40.3 mm to (126.0, 52.4)
- moved U1 40.3 mm to (154.2, 57.6)
- moved BOOT1 40.3 mm to (178.3, 81.7)
- moved C1 40.3 mm to (138.9, 49.5)
- moved C2 40.3 mm to (132.4, 49.5)
- moved C4 40.3 mm to (168.9, 66.0)
- moved RESET1 40.3 mm to (129.9, 82.0)
Other:
- board size 66 x 132.5 mm -> 115 x 100 mm
- board text added: "Bas"
- board text added: "Haut"
Changed lines of the file:
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@@
 		(tags "capacitor")
 		(property "Reference" "C6"
-			(at 0 -1.68 360)
+			(at 0 -1.68 0)
 			(layer "F.SilkS")
 			(effects
@@
 		)
 		(property "Value" "10µF"
-			(at 0 1.68 360)
+			(at 0 1.68 0)
 			(layer "F.Fab")
 			(effects
@@
 		)
 		(fp_text user "${REFERENCE}"
-			(at 0 0 360)
+			(at 0 0 0)
 			(layer "F.Fab")
 			(effects
@@
 	(footprint "Capacitor_SMD:C_0805_2012Metric"
 		(layer "F.Cu")
-		(at 134 86)
+		(at 168.95 65.95)
 		(descr "Capacitor SMD 0805 (2012 Metric), square (rectangular) end terminal, IPC_7351 nominal, (Body size source: IPC-SM-782 page 76, https://www.pcb-3d.com/wordpress/wp-content/uploads/ipc-sm-782a_amendment_1_and_2.pdf, https://docs.google.com/spreadsheets/d/1BsfQQcO9C6DZCsRaXUlFlo91Tg2WpOkGARC1WS5S8t0/edit?usp=sharing), generated with kicad-footprint-generator")
 		(tags "capacitor")
@@
 	(footprint "Capacitor_SMD:C_0805_2012Metric"
 		(layer "F.Cu")
-		(at 91 72.45 90)
+		(at 125.95 52.4 90)
 		(descr "Capacitor SMD 0805 (2012 Metric), square (rectangular) end terminal, IPC_7351 nominal, (Body size source: IPC-SM-782 page 76, https://www.pcb-3d.com/wordpress/wp-content/uploads/ipc-sm-782a_amendment_1_and_2.pdf, https://docs.google.com/spreadsheets/d/1BsfQQcO9C6DZCsRaXUlFlo91Tg2WpOkGARC1WS5S8t0/edit?usp=sharing), generated with kicad-footprint-generator")
 		(tags "capacitor")
@@
 	(footprint "Button_Switch_SMD:SW_MEC_5GSH9"
 		(layer "F.Cu")
-		(at 95 102 180)
+		(at 129.95 81.95 180)
 		(descr "MEC 5G single pole normally-open tactile switch")
 		(tags "switch normally-open pushbutton push-button")
 		(property "Reference" "RESET1"
-			(at -3.325 -8.575 360)
+			(at -3.325 -8.575 0)
 			(layer "F.SilkS")
 			(effects
@@
 		)
 		(property "Value" "SW_MEC_5E"
-			(at 0.475 8.825 360)
+			(at 0.475 8.825 0)
 			(layer "F.Fab")
 			(effects
@@
 		)
 		(fp_text user "${REFERENCE}"
-			(at 0 0 360)
+			(at 0 0 0)
 			(layer "F.Fab")
 			(effects
@@
 	(footprint "Capacitor_SMD:C_0805_2012Metric"
 		(layer "F.Cu")
-		(at 104 69.5 90)
+		(at 138.95 49.45 90)
 		(descr "Capacitor SMD 0805 (2012 Metric), square (rectangular) end terminal, IPC_7351 nominal, (Body size source: IPC-SM-782 page 76, https://www.pcb-3d.com/wordpress/wp-content/uploads/ipc-sm-782a_amendment_1_and_2.pdf, https://docs.google.com/spreadsheets/d/1BsfQQcO9C6DZCsRaXUlFlo91Tg2WpOkGARC1WS5S8t0/edit?usp=sharing), generated with kicad-footprint-generator")
 		(tags "capacitor")
@@
 	(footprint "Button_Switch_SMD:SW_MEC_5GSH9"
 		(layer "F.Cu")
-		(at 143.31 101.75 180)
+		(at 178.26 81.7 180)
 		(descr "MEC 5G single pole normally-open tactile switch")
 		(tags "switch normally-open pushbutton push-button")
 		(property "Reference" "BOOT1"
-			(at -3.325 -8.575 360)
+			(at -3.325 -8.575 0)
 			(layer "F.SilkS")
 			(effects
@@
 		)
 		(property "Value" "SW_MEC_5E"
-			(at 0.475 8.825 360)
+			(at 0.475 8.825 0)
 			(layer "F.Fab")
 			(effects
@@
 		)
 		(fp_text user "${REFERENCE}"
-			(at 0 0 360)
+			(at 0 0 0)
 			(layer "F.Fab")
 			(effects
@@
 	(footprint "Capacitor_SMD:C_0805_2012Metric"
 		(layer "F.Cu")
-		(at 97.5 69.5 90)
+		(at 132.45 49.45 90)
 		(descr "Capacitor SMD 0805 (2012 Metric), square (rectangular) end terminal, IPC_7351 nominal, (Body size source: IPC-SM-782 page 76, https://www.pcb-3d.com/wordpress/wp-content/uploads/ipc-sm-782a_amendment_1_and_2.pdf, https://docs.google.com/spreadsheets/d/1BsfQQcO9C6DZCsRaXUlFlo91Tg2WpOkGARC1WS5S8t0/edit?usp=sharing), generated with kicad-footprint-generator")
 		(tags "capacitor")
@@
 		(tags "resistor")
 		(property "Reference" "R6"
-			(at 0 -1.65 360)
+			(at 0 -1.65 0)
 			(layer "F.SilkS")
 			(effects
@@
 		)
 		(property "Value" "1M"
-			(at 0 1.65 360)
+			(at 0 1.65 0)
 			(layer "F.Fab")
 			(effects
@@
 		)
 		(fp_text user "${REFERENCE}"
-			(at 0 0 360)
+			(at 0 0 0)
 			(layer "F.Fab")
 			(effects
@@
 	(footprint "RF_Module:ESP32-S3-WROOM-1U"
 		(layer "F.Cu")
-		(at 119.3 77.69)
+		(at 154.25 57.64)
 		(descr "2.4 GHz Wi-Fi and Bluetooth module  https://www.espressif.com/sites/default/files/documentation/esp32-s3-wroom-1_wroom-1u_datasheet_en.pdf")
 		(tags "2.4 GHz Wi-Fi and Bluetooth module")
@@
 		)
 		(fp_text user "${REFERENCE}"
-			(at 0 0 360)
+			(at 0 0 0)
 			(layer "F.Fab")
 			(effects
@@
 	(footprint "Resistor_SMD:R_0805_2012Metric"
 		(layer "F.Cu")
-		(at 98.4125 74.5)
+		(at 133.3625 54.45)
 		(descr "Resistor SMD 0805 (2012 Metric), square (rectangular) end terminal, IPC_7351 nominal, (Body size source: IPC-SM-782 page 72, https://www.pcb-3d.com/wordpress/wp-content/uploads/ipc-sm-782a_amendment_1_and_2.pdf), generated with kicad-footprint-generator")
 		(tags "resistor")
 		(property "Reference" "R3"
-			(at 0 -1.65 360)
+			(at 0 -1.65 0)
 			(layer "F.SilkS")
 			(effects
@@
 		)
 		(property "Value" "10k"
-			(at 0 1.65 360)
+			(at 0 1.65 0)
 			(layer "F.Fab")
 			(effects
@@
 		)
 		(fp_text user "${REFERENCE}"
-			(at 0 0 360)
+			(at 0 0 0)
 			(layer "F.Fab")
 			(effects
@@
 	)
 	(gr_rect
-		(start 85.5 37.5)
-		(end 151.5 170)
+		(start 85 50)
+		(end 200 150)
 		(stroke
 			(width 0.05)
@@
 		(layer "Edge.Cuts")
 	)
+	(gr_text "Haut"
+		(at 127 28.5 0)
+		(layer "Cmts.User")
+		(effects
+			(font
+				(size 5 5)
+				(thickness 0.15)
+			)
+			(justify left bottom)
+		)
+	)
+	(gr_text "Bas"
+		(at 126.5 189.5 0)
+		(layer "Cmts.User")
+		(effects
+			(font
+				(size 5 5)
+				(thickness 0.15)
+			)
+			(justify left bottom)
+		)
+	)
 )

Commit message: Mise à jour documents
Parts:
- added J2: Conn_Coaxial, Connector_Coaxial:SMA_Molex_73251-1153_EdgeMount_Horizontal, F.Cu at (184.3, 62.0)
- added U4: ESP32-S3-DevKitC, PCM_Espressif:ESP32-S3-DevKitC, F.Cu at (166.4, 111.1)
- moved J1 105.4 mm to (90.0, 61.0), turned to -90 degrees
- moved RESET1 104.8 mm to (36.4, 34.8)
- moved R3 85.5 mm to (56.8, 16.4)
- moved C1 85.5 mm to (62.4, 11.3)
- moved C2 85.5 mm to (55.9, 11.3)
- moved C3 85.5 mm to (49.4, 14.3)
- moved BOOT1 84.6 mm to (107.1, 36.0)
- moved U1 84.5 mm to (73.0, 34.6)
- moved C4 76.9 mm to (107.4, 19.8)
- moved R8 35.3 mm to (90.5, 144.3), turned to 90 degrees
- moved D2 33.7 mm to (90.5, 149.5), turned to 90 degrees
- moved C7 27.4 mm to (96.0, 145.3), turned to 90 degrees
- moved R7 23.2 mm to (101.0, 142.4), turned to 90 degrees
- moved R6 19.6 mm to (101.0, 147.8), turned to 90 degrees
- moved U3 9.01 mm to (109.5, 147.8), turned to 180 degrees
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Other:
- board size 115 x 100 mm -> 100 x 115 mm

Commit message: Update Kicad Schematic
Parts:
- removed BOOT1, RESET1: SW_MEC_5E, Button_Switch_SMD:SW_MEC_5GSH9
- removed C1, C3, C4: 0.1µF, Capacitor_SMD:C_0805_2012Metric
- removed C2, C6, C7: 10µF, Capacitor_SMD:C_0805_2012Metric
- removed J1: USB_C_Receptacle_USB2.0_16P, Connector_USB:USB_C_Receptacle_GCT_USB4085
- removed J2: Conn_Coaxial, Connector_Coaxial:SMA_Molex_73251-1153_EdgeMount_Horizontal
- removed R3: 10k, Resistor_SMD:R_0805_2012Metric
- removed R6: 1M, Resistor_SMD:R_0805_2012Metric
- removed R7: 200k, Resistor_SMD:R_0805_2012Metric
- removed R8: 5.1K, Resistor_SMD:R_0805_2012Metric
- removed U1: ESP32-S3-WROOM-1, RF_Module:ESP32-S3-WROOM-1U
- removed U2: D3V3XA4B10LP, Package_DFN_QFN:Diodes_UDFN-10_1.0x2.5mm_P0.5mm
- removed U3: TLV75801PDBV, Package_TO_SOT_SMD:SOT-23-5
- added D1: GREEN, LED_SMD:LED_1206_3216Metric, F.Cu at (91.0, 92.0)
- added FB1: FerriteBead, Ferrite_THT:LairdTech_28C0236-0JW-10, F.Cu at (106.9, 44.0)
- added J5: Conn_01x04_Socket, Connector_JST:JST_XH_B4B-XH-A_1x04_P2.50mm_Vertical, F.Cu at (103.5, 150.0)
- added Q1: MMBT3904, Package_TO_SOT_SMD:SOT-23, F.Cu at (86.9, 60.0)
- added R1: 330R, Resistor_SMD:R_1206_3216Metric, F.Cu at (104.5, 92.0)
- added R2: 330R, Resistor_SMD:R_1206_3216Metric, F.Cu at (104.5, 97.5)
- added SW1: REP TEST, Button_Switch_THT:SW_PUSH_6mm, F.Cu at (89.0, 106.0)
- D2: value LED -> RED; footprint LED_SMD:LED_0805_2012Metric -> LED_SMD:LED_1206_3216Metric
- moved U4 73.4 mm to (111.6, 62.2), turned to 0 degrees
- moved D2 52.0 mm to (91.1, 97.5), turned to 0 degrees
Connections:
- net Net-(U4-3V3-Pad1) renamed VCC
- U4 pad 15: unconnected-(U4-GPIO9/ADC1_CH8-Pad15) -> Net-(U4-GPIO9/ADC1_CH8)
- U4 pad 16: unconnected-(U4-GPIO10/ADC1_CH9-Pad16) -> Net-(U4-GPIO10/ADC1_CH9)
- U4 pad 17: unconnected-(U4-GPIO11/ADC2_CH0-Pad17) -> Net-(U4-GPIO11/ADC2_CH0)
- U4 pad 22: Net-(U4-GND-Pad22) -> GND
- U4 pad 23: Net-(U4-GND-Pad22) -> GND
- U4 pad 24: Net-(U4-GND-Pad22) -> GND
- U4 pad 44: Net-(U4-GND-Pad22) -> GND
